File: microcontroller.sch (KiCad schematic (older format))
At the start: 0 parts

Commit message: Add microcontroller
Parts:
- added C? (x3): C, symbol dmpro-rescue:C
- added J?: Conn_ARM_JTAG_SWD_20, symbol dmpro-rescue:Conn_ARM_JTAG_SWD_20
- added U?: EFM32GG942F1024, QFP64_10X10, symbol dmpro-rescue:EFM32GG942F1024
- added Y?: Crystal_GND24, symbol dmpro-rescue:Crystal_GND24
Connections:
- new net: J?.15 (~SRST~), U?.20 (RESETN)
- new net: C?.1, U?.24 (PB13), Y?.3
- new net: C?.1, U?.25 (PB14), Y?.1
- new net: C?.1, U?.40 (DECOUPLE)
- new net: J?.9 (TCK/SWDCLK), U?.49 (PF0)
- new net: J?.7 (TMS/SWDIO), U?.50 (PF1)
- new net: J?.13 (TDO/SWO), U?.51 (PF2)
- new net +3V3: U?.26 (IOVDD_3), U?.39 (VDD_DREG), U?.55 (IOVDD_5), U?.7 (IOVDD_0)
- new net GND: C?.2, C?.2, C?.2, J?.10 (GND), J?.12 (GND), J?.14 (GND), J?.16 (GND), J?.18 (GND), J?.20 (GND), J?.4 (GND), J?.6 (GND), J?.8 (GND), U?.22 (VSS), U?.56 (VSS), U?.8 (VSS), Y?.2, Y?.4
