File: audio.sch (KiCad schematic (older format))
At the start: 0 parts

Commit message: Progress on audio scheme
Parts:
- added C? (x3): 0.1u, symbol Device:C_Small
- added C? (x3): 10u, symbol Device:CP1_Small
- added C?: 1u, symbol Device:CP1_Small
- added C? (x5): 4.7u, symbol Device:CP1_Small
- added U?: PCM3003E, DB24, symbol pcm3003:PCM3003E
- added U?: DRV632PWR, PW14, symbol drv632:DRV632PWR
- added U?: INA1651IPW, PW0014A_N, symbol ina1651:INA1651IPW
Connections:
- new net: C?.1, C?.2
- new net: C?.1, U?.6 (VINL)
- new net: C?.2, U?.13 (OUTA)
- new net: C?.1, U?.19 (VOUTL)
- new net: C?.1, U?.20 (VOUTR)
- new net: C?.1, U?.21 (VCOM)
- new net: C?.1, U?.4 (VREF1)
- new net: C?.1, U?.5 (VREF2)
- new net: C?.2, C?.2 (x2)
- new net +3.3VA: C?.1, C?.1, C?.1, U?.1 (VCC1), U?.14 (VDD), U?.18 (DEM0), U?.2 (VCC1), U?.24 (VCC2), U?.7 (*PDAD), U?.8 (*PDDA)
- new net AudioIn+: U?.10 (VMID_OUT), U?.12 (REFA), U?.2 (+INA), U?.3 (COMA)
- new net AudioIn-: U?.4 (-INA)
- new net AudioOutL: C?.2
- new net AudioOutR: C?.2
- new net BITCLK: U?.11 (BCKIN)
- new net FPGAIn: U?.12 (DOUT)
- new net FPGAOut: U?.15 (DIN)
- new net GND: C?.1, C?.1, C?.2, C?.2, C?.2, C?.2, U?.13 (DGND), U?.17 (DEM1), U?.22 (AGND2), U?.23 (AGND1)
- new net LRCLK: U?.10 (LRCIN)
- new net SYSCLK: U?.9 (SYSCLK)

Commit message: More schemes
Parts:
- removed U?: DRV632PWR, PW14, symbol drv632:DRV632PWR
- added C? (x2): 10u, symbol Device:C_Small
- added C? (x2): 1u, symbol Device:C_Small
- added C?: 0.1u, symbol Device:C_Small
- added J?: AudioJack3_Ground, symbol Connector:AudioJack3_Ground
- added J? (x2): AudioJack2, symbol Connector:AudioJack2
- added R? (x2): 100k, symbol Device:R_Small
Connections:
- net GND: now also C?.2, U?.13 (OUTA), U?.14 (VEE), C?.1, C?.1, C?.2
- net +5VA: now reaches U?.1 (VCC)
- net +5VA: now also C?.1, C?.2
- net at U?.11 (VMID_IN): now also C?.2
- net AudioIn+: no longer names the net of U?.10 (VMID_OUT), U?.12 (REFA), U?.3 (COMA)
- net AudioIn+: no longer U?.2 (+INA)
- net AudioIn-: no longer names the net of U?.4 (-INA)
- net AudioIn-: now also C?.1
- net AudioOutL: no longer names the net of C?.2
- net AudioOutL: now also J?.T
- net AudioOutR: no longer names the net of C?.2
- net AudioOutR: now also J?.T
- new net: C?.1, U?.2 (+INA)
- new net: C?.2, J?.T, R?.1
- new net: J?.G, J?.S, R?.2, R?.2
- new net: C?.2, J?.R, R?.1
Other:
- moved on the sheet: C?, U?

Commit message: All the files
Parts:
- removed J?: AudioJack3_Ground, symbol Connector:AudioJack3_Ground
- removed J? (x2): AudioJack2, symbol Connector:AudioJack2
- added J? (x2): AudioJack3, symbol Connector:AudioJack3
Connections:
- net +3.3VA: now also C?.1, C?.2, C?.2
- net GND: now also C?.2, C?.2, C?.2, J?.S
- net at C?.1, U?.21 (VCOM): now also U?.3 (VINR)
- net at C?.2: now also J?.R
- net at C?.2: now also J?.T
- net at C?.2, R?.1: now also J?.T
- net at R?.2, R?.2: now also J?.S
- net at C?.2, R?.1: now also J?.R
- no-connect marks 0 -> 1
Other:
- moved on the sheet: C?
Changed lines of the file:
@@
 $Descr A3 16535 11693
 encoding utf-8
-Sheet 5 8
+Sheet 5 9
 Title ""
 Date ""
@@
 Connection ~ 11300 3300
 $Comp
-L Device:C_Small C?
-U 1 1 5D8A5F6F
-P 7150 3300
-F 0 "C?" V 6921 3300 50  0000 C CNN
-F 1 "0.1u" V 7012 3300 50  0000 C CNN
-F 2 "" H 7150 3300 50  0001 C CNN
-F 3 "~" H 7150 3300 50  0001 C CNN
-	1    7150 3300
-	0    1    1    0
-$EndComp
-$Comp
 L power:+3.3VA #PWR0141
 U 1 1 5D8D6997
@@
 Connection ~ 8400 3900
 Wire Wire Line
-	11650 3300 11750 3300
-Wire Wire Line
 	7600 3800 8500 3800
 $Comp
@@
 	12000 3500 12000 3600
 Wire Wire Line
-	11100 3600 11300 3600
-Wire Wire Line
 	11500 3600 12000 3600
 Wire Wire Line
@@
 $EndComp
 Wire Wire Line
-	7550 3300 8300 3300
+	7300 3300 7550 3300
 $Comp
 L Device:CP1_Small C?
 U 1 1 5D8A6788
-P 7450 3300
-F 0 "C?" V 7222 3300 50  0000 C CNN
-F 1 "10u" V 7313 3300 50  0000 C CNN
-F 2 "" H 7450 3300 50  0001 C CNN
-F 3 "~" H 7450 3300 50  0001 C CNN
-	1    7450 3300
-	0    1    1    0
-$EndComp
-Wire Wire Line
-	7350 3300 7250 3300
+P 7200 3300
+F 0 "C?" V 6972 3300 50  0000 C CNN
+F 1 "10u" V 7063 3300 50  0000 C CNN
+F 2 "" H 7200 3300 50  0001 C CNN
+F 3 "~" H 7200 3300 50  0001 C CNN
+	1    7200 3300
+	0    1    1    0
+$EndComp
 $Comp
 L power:GND #PWR0143
@@
 $EndComp
 Wire Wire Line
-	7050 3300 7050 3450
-Wire Wire Line
 	7850 3350 7850 3450
-Wire Wire Line
-	7050 3450 7850 3450
 Connection ~ 7050 3450
 Wire Wire Line
@@
 Connection ~ 11700 4600
 Wire Wire Line
-	11400 4600 11700 4600
+	11400 4600 11650 4600
 Wire Wire Line
 	11400 4000 11400 4600
@@
 $EndComp
 Wire Wire Line
-	11650 4450 11750 4450
-Wire Wire Line
 	11450 4450 11450 4300
 Wire Wire Line
 	11100 4300 11450 4300
 Wire Wire Line
-	11450 4300 12150 4300
+	11450 4300 11750 4300
 Connection ~ 11450 4300
 Wire Wire Line
@@
 	10650 2250 10650 2500
 Wire Wire Line
-	12000 3300 12350 3300
-Wire Wire Line
-	11300 2500 12150 2500
+	12000 3300 12100 3300
+Wire Wire Line
+	11300 2500 11750 2500
 Text GLabel 10350 5000 0    50   Input ~ 0
 FPGAOut
@@
 	6600 3100 5000 3100
 Connection ~ 6600 3700
-$Comp
-L Connector:AudioJack3_Ground J?
-U 1 1 5DB8BF0E
+Wire Wire Line
+	3300 4000 3300 4200
+Wire Wire Line
+	3300 4200 3450 4200
+Connection ~ 3450 4200
+Wire Wire Line
+	3300 3900 3750 3900
+Wire Wire Line
+	3750 3950 3750 3900
+Connection ~ 3750 3900
+Wire Wire Line
+	3750 3900 4000 3900
+Connection ~ 6600 3800
+$Comp
+L Connector:AudioJack3 J?
+U 1 1 5D92FF52
+P 13450 3750
+F 0 "J?" H 13170 3683 50  0000 R CNN
+F 1 "AudioJack3" H 13170 3774 50  0000 R CNN
+F 2 "" H 13450 3750 50  0001 C CNN
+F 3 "~" H 13450 3750 50  0001 C CNN
+	1    13450 3750
+	-1   0    0    1
+$EndComp
+Wire Wire Line
+	12900 3550 13000 3550
+Wire Wire Line
+	13000 3550 13000 3750
+Wire Wire Line
+	13000 3750 13250 3750
+Wire Wire Line
+	12900 3950 13100 3950
+Wire Wire Line
+	13100 3950 13100 3650
+Wire Wire Line
+	13100 3650 13250 3650
+Wire Wire Line
+	13250 3850 13250 4600
+Wire Wire Line
+	13250 4600 11950 4600
+Connection ~ 11950 4600
+$Comp
+L Connector:AudioJack3 J?
+U 1 1 5D973AB4
 P 3100 3900
-F 0 "J?" H 2821 3776 50  0000 R CNN
-F 1 "AudioJack3_Ground" H 2821 3867 50  0000 R CNN
+F 0 "J?" H 2821 3833 50  0000 R CNN
+F 1 "AudioJack3" H 2821 3924 50  0000 R CNN
 F 2 "" H 3100 3900 50  0001 C CNN
 F 3 "~" H 3100 3900 50  0001 C CNN
@@
 	1    0    0    1
 $EndComp
-Wire Wire Line
-	3300 4000 3300 4200
-Wire Wire Line
-	3300 4200 3450 4200
-Connection ~ 3300 4200
-Connection ~ 3450 4200
-Wire Wire Line
-	3300 3900 3750 3900
-Wire Wire Line
-	3750 3950 3750 3900
-Connection ~ 3750 3900
-Wire Wire Line
-	3750 3900 4000 3900
-Wire Wire Line
-	2650 4200 2650 3600
-Wire Wire Line
-	2650 3600 3100 3600
-Wire Wire Line
-	2650 4200 3300 4200
-$Comp
-L Connector:AudioJack2 J?
-U 1 1 5DC0ED03
-P 13500 3550
-F 0 "J?" H 13320 3625 50  0000 R CNN
-F 1 "AudioJack2" H 13320 3534 50  0000 R CNN
-F 2 "" H 13500 3550 50  0001 C CNN
-F 3 "~" H 13500 3550 50  0001 C CNN
-	1    13500 3550
-	-1   0    0    -1
-$EndComp
-$Comp
-L Connector:AudioJack2 J?
-U 1 1 5DC10832
-P 13500 3950
-F 0 "J?" H 13320 4025 50  0000 R CNN
-F 1 "AudioJack2" H 13320 3934 50  0000 R CNN
-F 2 "" H 13500 3950 50  0001 C CNN
-F 3 "~" H 13500 3950 50  0001 C CNN
-	1    13500 3950
-	-1   0    0    -1
-$EndComp
-Wire Wire Line
-	12900 3550 13300 3550
-Wire Wire Line
-	12900 3950 13300 3950
-Connection ~ 6600 3800
+NoConn ~ 11100 4100
+Wire Wire Line
+	11650 4450 11650 4600
+Connection ~ 11650 4600
+Wire Wire Line
+	11650 4600 11700 4600
+Wire Wire Line
+	11750 4450 11750 4300
+Connection ~ 11750 4300
+Wire Wire Line
+	11750 4300 12150 4300
+Wire Wire Line
+	11650 3300 11650 3050
+Wire Wire Line
+	11650 3050 12100 3050
+Wire Wire Line
+	12100 3050 12100 3300
+Connection ~ 12100 3300
+Wire Wire Line
+	12100 3300 12350 3300
+Wire Wire Line
+	11750 3300 11750 2500
+Connection ~ 11750 2500
+Wire Wire Line
+	11750 2500 12150 2500
+Wire Wire Line
+	7050 3450 7850 3450
+Wire Wire Line
+	11100 3600 11250 3600
+Wire Wire Line
+	8500 3500 8150 3500
+Wire Wire Line
+	8150 3500 8150 2850
+Wire Wire Line
+	8150 2850 11250 2850
+Wire Wire Line
+	11250 2850 11250 3600
+Connection ~ 11250 3600
+Wire Wire Line
+	11250 3600 11300 3600
+Wire Wire Line
+	7100 3300 7050 3300
+Connection ~ 7050 3300
+Wire Wire Line
+	7050 3300 7050 3450
+Wire Wire Line
+	7550 3100 7550 3300
+Connection ~ 7550 3300
+Wire Wire Line
+	7550 3300 8300 3300
+Wire Wire Line
+	7050 3100 7050 3300
+Wire Wire Line
+	7250 3100 7550 3100
+$Comp
+L Device:C_Small C?
+U 1 1 5D8A5F6F
+P 7150 3100
+F 0 "C?" V 6921 3100 50  0000 C CNN
+F 1 "0.1u" V 7012 3100 50  0000 C CNN
+F 2 "" H 7150 3100 50  0001 C CNN
+F 3 "~" H 7150 3100 50  0001 C CNN
+	1    7150 3100
+	0    1    1    0
+$EndComp
 Wire Wire Line
 	6600 3800 7400 3800
