File: audio.sch (KiCad schematic (older format))
At the start: 23 parts, among them J7 AudioJack3, J8 AudioJack3, U8 INA1651IPW, U9 PCM3003E

Commit message: Update annotations and footprints
Parts:
- C64, C65, C66, C67, C68, C69, C70, C71, C72, C73, C74, C75, C76, C77, C78, C79, C80: footprint (none) -> Capacitor_SMD:C_1206_3216Metric_Pad1.42x1.75mm_HandSolder
- R18, R19: footprint (none) -> Resistor_SMD:R_1206_3216Metric_Pad1.42x1.75mm_HandSolder
Changed lines of the file:
@@
 F 0 "C71" V 7272 3800 50  0000 C CNN
 F 1 "1u" V 7363 3800 50  0000 C CNN
-F 2 "" H 7500 3800 50  0001 C CNN
+F 2 "Capacitor_SMD:C_1206_3216Metric_Pad1.42x1.75mm_HandSolder" H 7500 3800 50  0001 C CNN
 F 3 "~" H 7500 3800 50  0001 C CNN
 	1    7500 3800
@@
 F 0 "C72" V 7722 3350 50  0000 C CNN
 F 1 "4.7u" V 7813 3350 50  0000 C CNN
-F 2 "" H 7950 3350 50  0001 C CNN
+F 2 "Capacitor_SMD:C_1206_3216Metric_Pad1.42x1.75mm_HandSolder" H 7950 3350 50  0001 C CNN
 F 3 "~" H 7950 3350 50  0001 C CNN
 	1    7950 3350
@@
 F 0 "C73" V 7722 3700 50  0000 C CNN
 F 1 "4.7u" V 7813 3700 50  0000 C CNN
-F 2 "" H 7950 3700 50  0001 C CNN
+F 2 "Capacitor_SMD:C_1206_3216Metric_Pad1.42x1.75mm_HandSolder" H 7950 3700 50  0001 C CNN
 F 3 "~" H 7950 3700 50  0001 C CNN
 	1    7950 3700
@@
 F 0 "C77" V 11621 3300 50  0000 C CNN
 F 1 "0.1u" V 11712 3300 50  0000 C CNN
-F 2 "" H 11850 3300 50  0001 C CNN
+F 2 "Capacitor_SMD:C_1206_3216Metric_Pad1.42x1.75mm_HandSolder" H 11850 3300 50  0001 C CNN
 F 3 "~" H 11850 3300 50  0001 C CNN
 	1    11850 3300
@@
 F 0 "C75" V 11778 3300 50  0000 C CNN
 F 1 "10u" V 11687 3300 50  0000 C CNN
-F 2 "" H 11550 3300 50  0001 C CNN
+F 2 "Capacitor_SMD:C_1206_3216Metric_Pad1.42x1.75mm_HandSolder" H 11550 3300 50  0001 C CNN
 F 3 "~" H 11550 3300 50  0001 C CNN
 	1    11550 3300
@@
 F 0 "C74" V 11628 3600 50  0000 C CNN
 F 1 "4.7u" V 11537 3600 50  0000 C CNN
-F 2 "" H 11400 3600 50  0001 C CNN
+F 2 "Capacitor_SMD:C_1206_3216Metric_Pad1.42x1.75mm_HandSolder" H 11400 3600 50  0001 C CNN
 F 3 "~" H 11400 3600 50  0001 C CNN
 	1    11400 3600
@@
 F 0 "C70" V 6972 3300 50  0000 C CNN
 F 1 "10u" V 7063 3300 50  0000 C CNN
-F 2 "" H 7200 3300 50  0001 C CNN
+F 2 "Capacitor_SMD:C_1206_3216Metric_Pad1.42x1.75mm_HandSolder" H 7200 3300 50  0001 C CNN
 F 3 "~" H 7200 3300 50  0001 C CNN
 	1    7200 3300
@@
 F 0 "C78" V 12021 4450 50  0000 C CNN
 F 1 "0.1u" V 12112 4450 50  0000 C CNN
-F 2 "" H 12250 4450 50  0001 C CNN
+F 2 "Capacitor_SMD:C_1206_3216Metric_Pad1.42x1.75mm_HandSolder" H 12250 4450 50  0001 C CNN
 F 3 "~" H 12250 4450 50  0001 C CNN
 	1    12250 4450
@@
 F 0 "C79" V 13028 3550 50  0000 C CNN
 F 1 "4.7u" V 12937 3550 50  0000 C CNN
-F 2 "" H 12800 3550 50  0001 C CNN
+F 2 "Capacitor_SMD:C_1206_3216Metric_Pad1.42x1.75mm_HandSolder" H 12800 3550 50  0001 C CNN
 F 3 "~" H 12800 3550 50  0001 C CNN
 	1    12800 3550
@@
 F 0 "C80" V 13028 3950 50  0000 C CNN
 F 1 "4.7u" V 12937 3950 50  0000 C CNN
-F 2 "" H 12800 3950 50  0001 C CNN
+F 2 "Capacitor_SMD:C_1206_3216Metric_Pad1.42x1.75mm_HandSolder" H 12800 3950 50  0001 C CNN
 F 3 "~" H 12800 3950 50  0001 C CNN
 	1    12800 3950
@@
 F 0 "R18" H 3509 4096 50  0000 L CNN
 F 1 "100k" H 3509 4005 50  0000 L CNN
-F 2 "" H 3450 4050 50  0001 C CNN
+F 2 "Resistor_SMD:R_1206_3216Metric_Pad1.42x1.75mm_HandSolder" H 3450 4050 50  0001 C CNN
 F 3 "~" H 3450 4050 50  0001 C CNN
 	1    3450 4050
@@
 F 0 "R19" H 3809 4096 50  0000 L CNN
 F 1 "100k" H 3809 4005 50  0000 L CNN
-F 2 "" H 3750 4050 50  0001 C CNN
+F 2 "Resistor_SMD:R_1206_3216Metric_Pad1.42x1.75mm_HandSolder" H 3750 4050 50  0001 C CNN
 F 3 "~" H 3750 4050 50  0001 C CNN
 	1    3750 4050
@@
 F 0 "C64" V 3721 3800 50  0000 C CNN
 F 1 "10u" V 3812 3800 50  0000 C CNN
-F 2 "" H 3950 3800 50  0001 C CNN
+F 2 "Capacitor_SMD:C_1206_3216Metric_Pad1.42x1.75mm_HandSolder" H 3950 3800 50  0001 C CNN
 F 3 "~" H 3950 3800 50  0001 C CNN
 	1    3950 3800
@@
 F 0 "C65" V 3871 3900 50  0000 C CNN
 F 1 "10u" V 3962 3900 50  0000 C CNN
-F 2 "" H 4100 3900 50  0001 C CNN
+F 2 "Capacitor_SMD:C_1206_3216Metric_Pad1.42x1.75mm_HandSolder" H 4100 3900 50  0001 C CNN
 F 3 "~" H 4100 3900 50  0001 C CNN
 	1    4100 3900
@@
 F 0 "C68" H 6692 3946 50  0000 L CNN
 F 1 "1u" H 6692 3855 50  0000 L CNN
-F 2 "" H 6600 3900 50  0001 C CNN
+F 2 "Capacitor_SMD:C_1206_3216Metric_Pad1.42x1.75mm_HandSolder" H 6600 3900 50  0001 C CNN
 F 3 "~" H 6600 3900 50  0001 C CNN
 	1    6600 3900
@@
 F 0 "C66" V 4471 2700 50  0000 C CNN
 F 1 "1u" V 4562 2700 50  0000 C CNN
-F 2 "" H 4700 2700 50  0001 C CNN
+F 2 "Capacitor_SMD:C_1206_3216Metric_Pad1.42x1.75mm_HandSolder" H 4700 2700 50  0001 C CNN
 F 3 "~" H 4700 2700 50  0001 C CNN
 	1    4700 2700
@@
 F 0 "C67" V 4929 3100 50  0000 C CNN
 F 1 "0.1u" V 4838 3100 50  0000 C CNN
-F 2 "" H 4700 3100 50  0001 C CNN
+F 2 "Capacitor_SMD:C_1206_3216Metric_Pad1.42x1.75mm_HandSolder" H 4700 3100 50  0001 C CNN
 F 3 "~" H 4700 3100 50  0001 C CNN
 	1    4700 3100
@@
 F 0 "C69" V 6971 2900 50  0000 C CNN
 F 1 "0.1u" V 7062 2900 50  0000 C CNN
-F 2 "" H 7200 2900 50  0001 C CNN
+F 2 "Capacitor_SMD:C_1206_3216Metric_Pad1.42x1.75mm_HandSolder" H 7200 2900 50  0001 C CNN
 F 3 "~" H 7200 2900 50  0001 C CNN
 	1    7200 2900
@@
 F 0 "C76" V 12028 4450 50  0000 C CNN
 F 1 "10u" V 11937 4450 50  0000 C CNN
-F 2 "" H 11800 4450 50  0001 C CNN
+F 2 "Capacitor_SMD:C_1206_3216Metric_Pad1.42x1.75mm_HandSolder" H 11800 4450 50  0001 C CNN
 F 3 "~" H 11800 4450 50  0001 C CNN
 	1    11800 4450

Commit message: Minor unrelated fixes
Parts:
- U9: footprint DB24 -> Package_SO:SSOP-24_5.3x8.2mm_P0.65mm
Changed lines of the file:
@@
 F 0 "U9" H 9800 3687 60  0000 C CNN
 F 1 "PCM3003E" H 9800 3581 60  0000 C CNN
-F 2 "DB24" H 9800 3540 60  0001 C CNN
+F 2 "Package_SO:SSOP-24_5.3x8.2mm_P0.65mm" H 9800 3540 60  0001 C CNN
 F 3 "" H 8500 3300 60  0000 C CNN
 	1    8500 3300

Commit message: Fix all footprints
Parts:
- U8: footprint PW0014A_N -> Package_SO:TSSOP-14_4.4x5mm_P0.65mm
Changed lines of the file:
@@
 F 0 "U8" H 5400 4087 60  0000 C CNN
 F 1 "INA1651IPW" H 5400 3981 60  0000 C CNN
-F 2 "PW0014A_N" H 5400 3940 60  0001 C CNN
+F 2 "Package_SO:TSSOP-14_4.4x5mm_P0.65mm" H 5400 3940 60  0001 C CNN
 F 3 "" H 4400 3700 60  0000 C CNN
 	1    4400 3700
