File: audio2.sch (KiCad schematic (older format))
At the start: 15 parts

Commit message: All the files
Changed lines of the file:
@@
 $Descr A4 11693 8268
 encoding utf-8
-Sheet 6 8
+Sheet 6 9
 Title ""
 Date ""
@@
 F1 "audio_common.sch" 50
 $EndSheet
+$Sheet
+S 6400 4900 2450 800
+U 5D90AE9B
+F0 "audio_opamp" 50
+F1 "audio_opamp.sch" 50
+$EndSheet
 $EndSCHEMATC
